File: jtag_shield.sch (KiCad schematic (older format))
At the start: 8 parts, among them J1 AVR-JTAG-10, J2 AVR-ISP-6, Q1 BF245A

Commit message: Updated with changes from Magnus
Parts:
- added C1: 100n, Capacitors_THT:C_Disc_D5.1mm_W3.2mm_P5.00mm, symbol C
- added R3: 47k, Resistors_THT:R_Axial_DIN0207_L6.3mm_D2.5mm_P10.16mm_Horizontal, symbol R
Connections:
- wire segments 46 -> 50
Other:
- note added: "5V SUPPLY"
- note added: "AD4 to AD7 are not available \nwhen JTAG is enabled"
- note added: "Application note: \n\nJTAG setup\n- Cut the RESET-EN connection to disable Auto-reset (2mm-jumper recommended)\n- Program the JTAGEN fuse to enable the JTAG test access port/TAP"
- note added: "JTAG ACTIVITY"
- moved on the sheet: D1, R1
